Commit message: spawned arm in world, joint origin repositioning pending

File: urdf/dofbot.urdf (robot description, URDF)
Before this commit: robot arm, 6 links, 5 joints
Links:
- link base_link: geometry collision mesh filename=package://robotic-arm-refuelling/meshes/base_link.STL scale=5 5 5; visual mesh filename=package://robotic-arm-refuelling/meshes/base_link.STL scale=5 5 5
- link link1: mass None -> 10; geometry collision mesh filename=package://robotic-arm-refuelling/meshes/link1.STL scale=5 5 5; visual mesh filename=package://robotic-arm-refuelling/meshes/link1.STL scale=5 5 5
- link link2: mass None -> 10; geometry collision mesh filename=package://robotic-arm-refuelling/meshes/link2.STL scale=5 5 5; visual mesh filename=package://robotic-arm-refuelling/meshes/link2.STL scale=5 5 5
- link link3: mass None -> 10; geometry collision mesh filename=package://robotic-arm-refuelling/meshes/link3.STL scale=5 5 5; visual mesh filename=package://robotic-arm-refuelling/meshes/link3.STL scale=5 5 5
- link link4: mass None -> 10; geometry collision mesh filename=package://robotic-arm-refuelling/meshes/link4.STL scale=5 5 5; visual mesh filename=package://robotic-arm-refuelling/meshes/link4.STL scale=5 5 5
- link link5: mass None -> 10; geometry collision mesh filename=package://robotic-arm-refuelling/meshes/link5.STL scale=5 5 5; visual mesh filename=package://robotic-arm-refuelling/meshes/link5.STL scale=5 5 5

Commit message: arm ready, to be repositioned

File: urdf/dofbot.urdf (robot description, URDF)
Before this commit: robot arm, 6 links, 5 joints
Links:
- link base_link: mass None -> 100
Joints:
- joint joint1: origin xyz=0 0 0.06605 rpy=-0.010805 0 0 -> xyz=0 0 0.33025 rpy=-0.010805 0 0
- joint joint2: origin xyz=0 -0.00031873 0.04145 rpy=0 1.5708 0 -> xyz=0 -0.00159365 0.20725 rpy=0 1.5708 0
- joint joint3: origin xyz=-0.08285 0 0 rpy=0 0 0 -> xyz=-0.41425 0 0 rpy=0 0 0
- joint joint4: origin xyz=-0.08285 0 0 rpy=0 0 0.0083081 -> xyz=-0.41425 0 0 rpy=0 0 0.0083081
- joint joint5: origin xyz=-0.07385 -0.001 0 rpy=0 -1.57 0 -> xyz=-0.36925 -0.005 0 rpy=0 -1.57 0

Commit message: arm ready with injector, UGV with receptacle pending.

File: urdf/dofbot.urdf (robot description, URDF)
Before this commit: robot arm, 6 links, 5 joints
Links:
- link base_link: mass 100 -> 10
- link link5: geometry collision mesh filename=package://robotic-arm-refuelling/meshes/injector.STL scale=0.003 0.003 0.003; visual mesh filename=package://robotic-arm-refuelling/meshes/injector.STL scale=0.003 0.003 0.003

Commit message: car files imported, multi robot launch problems need fixing
changes since last commit :
- new committing standard
- world file finished
- dofbot with male injector completed and placed
- joint trajectory controller implemented

near term features pending (deadline - 16th June, 2023) :
- car urdf modified with female component and visual odometry pattern
- car controller
- demo scripts for static refuelling with cvbridge
- new car urdf with arm & male connector
- adjust inertia values for dofbot components
- testing to collect data for static refuelling (write nodes)
    - time for refuelling
    - payload capacity
    - end effector details
    - arm velocity
    - edge detections
    - docking and undocking time
    - alignment accuracy while docking (x, y, z)

long term features pending :
- demo scripts for dynamic refuelling
- patent & publication writing
- multidimensional synchronization for dynamic case (tbd)
- in-space arm docking (tbd)

current commit policy - commit to main

File: urdf/dofbot.urdf (robot description, URDF)
Before this commit: robot arm, 6 links, 5 joints
Links:
- link base_link: geometry collision mesh filename=package://robotic-arm-refuelling/meshes/dofbot/base_link.STL scale=5 5 5; visual mesh filename=package://robotic-arm-refuelling/meshes/dofbot/base_link.STL scale=5 5 5
- link link1: geometry collision mesh filename=package://robotic-arm-refuelling/meshes/dofbot/link1.STL scale=5 5 5; visual mesh filename=package://robotic-arm-refuelling/meshes/dofbot/link1.STL scale=5 5 5
- link link2: geometry collision mesh filename=package://robotic-arm-refuelling/meshes/dofbot/link2.STL scale=5 5 5; visual mesh filename=package://robotic-arm-refuelling/meshes/dofbot/link2.STL scale=5 5 5
- link link3: geometry collision mesh filename=package://robotic-arm-refuelling/meshes/dofbot/link3.STL scale=5 5 5; visual mesh filename=package://robotic-arm-refuelling/meshes/dofbot/link3.STL scale=5 5 5
- link link4: geometry collision mesh filename=package://robotic-arm-refuelling/meshes/dofbot/link4.STL scale=5 5 5; visual mesh filename=package://robotic-arm-refuelling/meshes/dofbot/link4.STL scale=5 5 5
- link link5: geometry collision mesh filename=package://robotic-arm-refuelling/meshes/refueller/injector.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 scale=0.003 0.003 0.003; visual mesh filename=package://robotic-arm-refuelling/meshes/refueller/injector.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 scale=0.003 0.003 0.003
