Commit message: arm and car spawned, camera plugin installed
changes since last commit :
- multi robot spawning fixed
- camera plugin issues solved
- camera aligned

near term features pending (deadline - 16th June, 2023) :
- inertia for dofbot to be tuned and/or new arm to be tuned and used
- car urdf modified with female component and visual odometry pattern
- car controller
- demo scripts for static refuelling with cvbridge
- new car urdf with arm & male connector
- adjust inertia values for dofbot components
- testing to collect data for static refuelling (write nodes)
    - time for refuelling
    - payload capacity
    - end effector details
    - arm velocity
    - edge detections
    - docking and undocking time
    - alignment accuracy while docking (x, y, z)

long term features pending :
- demo scripts for dynamic refuelling
- patent & publication writing
- multidimensional synchronization for dynamic case (tbd)
- in-space arm docking (tbd)

current commit policy - commit to main

File: urdf/arm/dofbot.urdf.xacro (robot description, xacro)
@@ -136,9 +136,8 @@
     <link name="camera_link_optical"></link>
     <joint name="camera_optical_joint" type="fixed">
-        <origin xyz="0 0 0" rpy="${-pi/2} 0 ${-pi/2}" />
+        <origin xyz="-0.33 -0.29 0" rpy="${-pi/2} 0 ${-pi}" />
         <parent link="link4" />
         <child link="camera_link_optical" />
     </joint>
-    <!-- link5 -->
     <link name="link5">
         <visual>
@@ -242,5 +241,5 @@
         <plugin name="control" filename="libgazebo_ros_control.so"/>
     </gazebo>
-    <gazebo reference="link4">
+    <gazebo reference="camera_link_optical">
         <sensor name="camera" type="camera">
             <pose> 0 0 0 0 0 0 </pose>
