Commit message: car files imported, multi robot launch problems need fixing
changes since last commit :
- new committing standard
- world file finished
- dofbot with male injector completed and placed
- joint trajectory controller implemented

near term features pending (deadline - 16th June, 2023) :
- car urdf modified with female component and visual odometry pattern
- car controller
- demo scripts for static refuelling with cvbridge
- new car urdf with arm & male connector
- adjust inertia values for dofbot components
- testing to collect data for static refuelling (write nodes)
    - time for refuelling
    - payload capacity
    - end effector details
    - arm velocity
    - edge detections
    - docking and undocking time
    - alignment accuracy while docking (x, y, z)

long term features pending :
- demo scripts for dynamic refuelling
- patent & publication writing
- multidimensional synchronization for dynamic case (tbd)
- in-space arm docking (tbd)

current commit policy - commit to main

File: urdf/arm/arm.urdf.xacro (robot description, xacro)
@@ -1,3 +1,4 @@
 <?xml version="1.0"?>
+<!--links misplaced, buggy-->
 <robot name="arm">
     <link name="world"/>
@@ -141,5 +142,5 @@
         </inertial>
         <visual>
-            <origin xyz="-0.3 0.1 0.1" rpy="0 0 0"/>
+            <origin xyz="-0.3 0.2 0.1" rpy="0 0 0"/>
             <geometry>
                 <box size="0.1 0.1 0.1"/>

File: urdf/arm/dofbot.urdf.xacro (robot description, xacro)
@@ -133,4 +133,10 @@
         <axis xyz="0 0 1" />
         <limit effort="30" velocity="1.0" lower="-1.5708" upper="1.5708"/>
+    </joint>
+    <link name="camera_link_optical"></link>
+    <joint name="camera_optical_joint" type="fixed">
+        <origin xyz="0 0 0" rpy="${-pi/2} 0 ${-pi/2}" />
+        <parent link="link4" />
+        <child link="camera_link_optical" />
     </joint>
     <!-- link5 -->
@@ -236,3 +242,25 @@
         <plugin name="control" filename="libgazebo_ros_control.so"/>
     </gazebo>
+    <gazebo reference="link4">
+        <sensor name="camera" type="camera">
+            <pose> 0 0 0 0 0 0 </pose>
+            <visualize>true</visualize>
+            <update_rate>10</update_rate>
+            <camera>
+                <horizontal_fov>1.089</horizontal_fov>
+                <image>
+                    <format>R8G8B8</format>
+                    <width>640</width>
+                    <height>480</height>
+                </image>
+                <clip>
+                    <near>0.05</near>
+                    <far>8.0</far>
+                </clip>
+            </camera>
+            <plugin name="camera_controller" filename="libgazebo_ros_camera.so">
+                <frame_name>camera_link_optical</frame_name>
+            </plugin>
+        </sensor>
+    </gazebo>
 </robot>

Commit message: joint trajectory controller implemented for arm, car urdf modified with receptacle
changes since last commit :
- joint trajectory controller for 5 dof arm completed
- inertia new arm to be tuned and used
- car urdf modified with female component and visual odometry pattern

near term features pending (deadline - 16th June, 2023) :
- inertia for dofbot to be tuned and used
- car controller
- demo scripts for static refuelling with cvbridge
- new car urdf with arm & male connector
- adjust inertia values for dofbot components
- testing to collect data for static refuelling (write nodes)
    - time for refuelling
    - payload capacity
    - end effector details
    - arm velocity
    - edge detections
    - docking and undocking time
    - alignment accuracy while docking (x, y, z)

long term features pending :
- demo scripts for dynamic refuelling
- patent & publication writing
- multidimensional synchronization for dynamic case (tbd)
- in-space arm docking (tbd)

current commit policy - commit to main

File: urdf/arm/arm.urdf.xacro (robot description, xacro)
@@ -1,4 +1,3 @@
 <?xml version="1.0"?>
-<!--links misplaced, buggy-->
 <robot name="arm">
     <link name="world"/>
@@ -135,34 +134,9 @@
         <origin rpy="0 0 0" xyz="0.0 0.1 0.35"/>
     </joint>
-    <link name="camera_link">
-        <inertial>
-            <origin xyz="-0.3 0.1 0.1" rpy="0 0 0"/>
-            <mass value="1"/>
-            <inertia ixx="0.00167" ixy="0.0" ixz="0.0" iyy="0.00167" iyz="0.0" izz="0.00167"/>
-        </inertial>
-        <visual>
-            <origin xyz="-0.3 0.2 0.1" rpy="0 0 0"/>
-            <geometry>
-                <box size="0.1 0.1 0.1"/>
-            </geometry>
-            <material name="red"/>
-        </visual>
-        <collision>
-            <origin xyz="-0.3 0.1 0.1" rpy="0 0 0"/>
-            <geometry>
-                <box size="0.1 0.1 0.1"/>
-            </geometry>
-        </collision>
-    </link>
+    <link name="camera_link"></link>
     <joint name="camera_joint" type="fixed">
         <parent link="link_4"/>
         <child link="camera_link"/>
-        <origin xyz="0.305 0 0.08" rpy="1.57 -1.57 0"/>
-    </joint>
-    <link name="camera_link_optical"></link>
-    <joint name="camera_optical_joint" type="fixed">
-        <origin xyz="0 0 0" rpy="${-pi/2} 0 ${-pi/2}" />
-        <parent link="camera_link" />
-        <child link="camera_link_optical" />
+        <origin xyz="0 0 0.55" rpy="1.57 -1.57 0"/>
     </joint>
     <link name="link_5">

File: urdf/car/car.xacro (robot description, xacro)
@@ -12,5 +12,5 @@
 	<xacro:property name="camera_mass" value="0.1"/>
 	<xacro:property name="hokoyu_mass" value="1e-5"/>
-	<!-- Make Chassis of Bot -->
+	<!-- Chassis -->
 	<link name="chassis">
 		<pose>0 0 0.1 0 0 0</pose>
@@ -37,4 +37,48 @@
 		</visual>
 	</link>
+	<!-- Fuel Inlet 1 -->
+	<link name="fuel_inlet1">
+        <visual>
+            <origin xyz="-0.25 0 0.15" rpy="-0.785 0 0"/>
+            <geometry>
+                <mesh filename="package://robotic-arm-refuelling/meshes/refueller/receptacle.stl" scale="0.003 0.003 0.003" />
+            </geometry>
+            <material name="">
+                <color rgba="1 1 1 1" />
+            </material>
+        </visual>
+        <collision>
+            <origin xyz="-0.25 0 0.15" rpy="-0.785 0 0"/>
+            <geometry>
+                <mesh filename="package://robotic-arm-refuelling/meshes/refueller/receptacle.stl" scale="0.003 0.003 0.003" />
+            </geometry>
+        </collision>
+        <inertial>
+        <mass value="10"/>
+        <inertia ixx="0.4" ixy="0.0" ixz="0.0" iyy="0.4" iyz="0.0" izz="0.4"/>
+        </inertial>
+    </link>
+	<!-- Fuel Inlet 2 -->
+	<link name="fuel_inlet2">
+        <visual>
+            <origin xyz="-0.25 -0.1 0.06" rpy="0.785 0 0"/>
+            <geometry>
+                <mesh filename="package://robotic-arm-refuelling/meshes/refueller/receptacle.stl" scale="0.003 0.003 0.003" />
+            </geometry>
+            <material name="">
+                <color rgba="1 1 1 1" />
+            </material>
+        </visual>
+        <collision>
+            <origin xyz="-0.25 -0.1 0.06" rpy="0.785 0 0"/>
+            <geometry>
+                <mesh filename="package://robotic-arm-refuelling/meshes/refueller/receptacle.stl" scale="0.003 0.003 0.003" />
+            </geometry>
+        </collision>
+        <inertial>
+        <mass value="10"/>
+        <inertia ixx="0.4" ixy="0.0" ixz="0.0" iyy="0.4" iyz="0.0" izz="0.4"/>
+        </inertial>
+    </link>
 	<!-- Right Wheel Back -->
 	<link name="right_wheel_back">
@@ -208,4 +252,18 @@
 		<child link="chassis" />
 	</joint>
+	<!-- Fuel Inlet Joint 1 -->
+	<joint name="fuel_joint1" type="fixed">
+        <origin xyz="0 0 0" rpy="0 0 0"/>
+        <axis xyz="0 0 1"/>
+        <parent link="chassis"/>
+        <child link="fuel_inlet1"/>
+    </joint>
+	<!-- Fuel Inlet Joint 2 -->
+	<joint name="fuel_joint2" type="fixed">
+        <origin xyz="0 0 0" rpy="0 0 0"/>
+        <axis xyz="0 0 1"/>
+        <parent link="chassis"/>
+        <child link="fuel_inlet2"/>
+    </joint>
 	<!-- Color of bot -->
 	<gazebo reference="left_wheel_front">
@@ -255,4 +313,62 @@
 	</gazebo>
 	<!-- Motor, Camera and Lidar Simulation -->
-	<xacro:include filename="$(find robotic-arm-refuelling)/urdf/car/atom.gazebo" />
+	<gazebo>
+		<plugin name="skid_steer_drive_controller" filename="libgazebo_ros_skid_steer_drive.so">
+			<updateRate>10.0</updateRate>
+			<robotNamespace>/atom</robotNamespace>
+			<leftFrontJoint>left_wheel_hinge_front</leftFrontJoint>
+			<rightFrontJoint>right_wheel_hinge_front</rightFrontJoint>
+			<leftRearJoint>left_wheel_hinge_back</leftRearJoint>
+			<rightRearJoint>right_wheel_hinge_back</rightRearJoint>
+			<wheelSeparation>0.4</wheelSeparation>
+			<wheelDiameter>0.2</wheelDiameter>
+			<robotBaseFrame>robot_footprint</robotBaseFrame>
+			<torque>10</torque>
+			<topicName>cmd_vel</topicName>
+			<odometryTopic>odom</odometryTopic>
+			<odometryFrame>odom</odometryFrame>
+			<commandTopic>cmd_vel</commandTopic>
+			<topic_name_twist>cmd_vel</topic_name_twist>
+			<topic_name_odometry>odom</topic_name_odometry>
+			<topic_name_joint>joint</topic_name_joint>
+			<broadcastTF>true</broadcastTF>
+			<covariance_x>0.0001</covariance_x>
+			<covariance_y>0.0001</covariance_y>
+			<covariance_yaw>0.01</covariance_yaw>
+		</plugin>
+	</gazebo>
+	<!-- camera -->
+	<gazebo reference="camera">
+		<sensor type="camera" name="camera1">
+			<visualize>true</visualize>
+			<update_rate>30.0</update_rate>
+			<camera name="head">
+				<horizontal_fov>1.3962634</horizontal_fov>
+				<image>
+				<width>800</width>
+				<height>800</height>
+				<format>R8G8B8</format>
+				</image>
+				<clip>
+				<near>0.02</near>
+				<far>300</far>
+				</clip>
+			</camera>
+			<plugin name="camera_controller" filename="libgazebo_ros_camera.so">
+				<robotNamespace>/atom</robotNamespace>
+				<alwaysOn>true</alwaysOn>
+				<updateRate>0.0</updateRate>
+				<cameraName>camera</cameraName>
+				<imageTopicName>rgb/image_raw</imageTopicName>
+				<cameraInfoTopicName>rgb/camera_info</cameraInfoTopicName>
+				<frameName>camera</frameName>
+				<hackBaseline>0.07</hackBaseline>
+				<distortionK1>0.0</distortionK1>
+				<distortionK2>0.0</distortionK2>
+				<distortionK3>0.0</distortionK3>
+				<distortionT1>0.0</distortionT1>
+				<distortionT2>0.0</distortionT2>
+			</plugin>
+		</sensor>
+  </gazebo>
 </robot>
